File: pathfinder/pathfinder.kicad_sch (KiCad schematic)
At the start: 10 parts, among them SW1 SW_Push, SW2 SW_Push, SW3 SW_Push, U1 XIAO-RP2040-DIP

Commit message: Started working on the PCB Editor
Parts:
- D1, D2, D3: footprint L08R5000Q1:LEDRD254W57D500H1070 -> footprints:LEDRD254W57D500H1070
- R1, R2, R3: footprint (none) -> Resistor_THT:R_Axial_DIN0204_L3.6mm_D1.6mm_P7.62mm_Horizontal
- SW1, SW2, SW3: footprint (none) -> Button_Switch_Keyboard:SW_Cherry_MX_1.00u_PCB
- U1: footprint Module:MOUDLE14P-XIAO-DIP-SMD -> footprints:XIAO-RP2040-DIP
Connections:
- net button1: now also SW1.1; no longer SW3.1
- net button2: now also SW2.1; no longer SW1.1
- net button3: now also SW3.1; no longer SW2.1
Changed lines of the file:
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@@
 	(global_label "button2"
 		(shape input)
-		(at 121.92 40.64 180)
+		(at 154.94 45.72 180)
 		(fields_autoplaced yes)
 		(effects
@@
 		)
 		(property "Intersheetrefs" "${INTERSHEET_REFS}"
-			(at 111.6779 40.64 0)
+			(at 144.6979 45.72 0)
 			(effects
 				(font
@@
 		)
 	)
-	(global_label "button3"
+	(global_label "LED3"
 		(shape input)
-		(at 154.94 45.72 180)
+		(at 154.94 76.2 180)
 		(fields_autoplaced yes)
 		(effects
@@
 		)
 		(property "Intersheetrefs" "${INTERSHEET_REFS}"
-			(at 144.6979 45.72 0)
+			(at 147.2982 76.2 0)
 			(effects
 				(font
@@
 	(global_label "button1"
 		(shape input)
-		(at 91.44 40.64 180)
+		(at 121.92 40.64 180)
 		(fields_autoplaced yes)
 		(effects
@@
 		)
 		(property "Intersheetrefs" "${INTERSHEET_REFS}"
-			(at 81.1979 40.64 0)
+			(at 111.6779 40.64 0)
 			(effects
 				(font
@@
 		)
 	)
-	(global_label "LED3"
+	(global_label "button1"
 		(shape input)
-		(at 154.94 76.2 180)
+		(at 113.03 96.52 180)
 		(fields_autoplaced yes)
 		(effects
@@
 		)
 		(property "Intersheetrefs" "${INTERSHEET_REFS}"
-			(at 147.2982 76.2 0)
+			(at 102.7879 96.52 0)
 			(effects
 				(font
@@
 		)
 	)
-	(global_label "button1"
+	(global_label "button3"
 		(shape input)
-		(at 113.03 96.52 180)
+		(at 113.03 104.14 180)
 		(fields_autoplaced yes)
 		(effects
@@
 		)
 		(property "Intersheetrefs" "${INTERSHEET_REFS}"
-			(at 102.7879 96.52 0)
+			(at 102.7879 104.14 0)
 			(effects
 				(font
@@
 		)
 	)
-	(global_label "button3"
+	(global_label "LED1"
 		(shape input)
-		(at 113.03 104.14 180)
+		(at 88.9 74.93 180)
 		(fields_autoplaced yes)
 		(effects
@@
 		)
 		(property "Intersheetrefs" "${INTERSHEET_REFS}"
-			(at 102.7879 104.14 0)
+			(at 81.2582 74.93 0)
 			(effects
 				(font
@@
 		)
 	)
-	(global_label "LED1"
+	(global_label "LED2"
 		(shape input)
-		(at 88.9 74.93 180)
+		(at 113.03 111.76 180)
 		(fields_autoplaced yes)
 		(effects
@@
 		)
 		(property "Intersheetrefs" "${INTERSHEET_REFS}"
-			(at 81.2582 74.93 0)
+			(at 105.3882 111.76 0)
 			(effects
 				(font
@@
 		)
 	)
-	(global_label "LED2"
+	(global_label "button2"
 		(shape input)
-		(at 113.03 111.76 180)
+		(at 113.03 100.33 180)
 		(fields_autoplaced yes)
 		(effects
@@
 		)
 		(property "Intersheetrefs" "${INTERSHEET_REFS}"
-			(at 105.3882 111.76 0)
+			(at 102.7879 100.33 0)
 			(effects
 				(font
@@
 		)
 	)
-	(global_label "button2"
+	(global_label "button3"
 		(shape input)
-		(at 113.03 100.33 180)
+		(at 91.44 40.64 180)
 		(fields_autoplaced yes)
 		(effects
@@
 		)
 		(property "Intersheetrefs" "${INTERSHEET_REFS}"
-			(at 102.7879 100.33 0)
+			(at 81.1979 40.64 0)
 			(effects
 				(font
@@
 			)
 		)
-		(property "Footprint" ""
+		(property "Footprint" "Resistor_THT:R_Axial_DIN0204_L3.6mm_D1.6mm_P7.62mm_Horizontal"
 			(at 153.162 72.39 90)
 			(effects
@@
 			)
 		)
-		(property "Footprint" ""
+		(property "Footprint" "Resistor_THT:R_Axial_DIN0204_L3.6mm_D1.6mm_P7.62mm_Horizontal"
 			(at 118.872 69.85 90)
 			(effects
@@
 			)
 		)
-		(property "Footprint" "L08R5000Q1:LEDRD254W57D500H1070"
+		(property "Footprint" "footprints:LEDRD254W57D500H1070"
 			(at 128.27 66.04 0)
 			(effects
@@
 			)
 		)
-		(property "Footprint" "L08R5000Q1:LEDRD254W57D500H1070"
+		(property "Footprint" "footprints:LEDRD254W57D500H1070"
 			(at 162.56 68.58 0)
 			(effects
@@
 			)
 		)
-		(property "Footprint" ""
+		(property "Footprint" "Button_Switch_Keyboard:SW_Cherry_MX_1.00u_PCB"
 			(at 160.02 40.64 0)
 			(effects
@@
 			)
 		)
-		(property "Footprint" ""
+		(property "Footprint" "Button_Switch_Keyboard:SW_Cherry_MX_1.00u_PCB"
 			(at 127 35.56 0)
 			(effects
@@
 			)
 		)
-		(property "Footprint" ""
+		(property "Footprint" "Button_Switch_Keyboard:SW_Cherry_MX_1.00u_PCB"
 			(at 96.52 35.56 0)
 			(effects
@@
 			)
 		)
-		(property "Footprint" ""
+		(property "Footprint" "Resistor_THT:R_Axial_DIN0204_L3.6mm_D1.6mm_P7.62mm_Horizontal"
 			(at 87.122 71.12 90)
 			(effects
@@
 			)
 		)
-		(property "Footprint" "Module:MOUDLE14P-XIAO-DIP-SMD"
+		(property "Footprint" "footprints:XIAO-RP2040-DIP"
 			(at 131.318 123.698 0)
 			(effects
@@
 			)
 		)
-		(property "Footprint" "L08R5000Q1:LEDRD254W57D500H1070"
+		(property "Footprint" "footprints:LEDRD254W57D500H1070"
 			(at 96.52 67.31 0)
 			(effects
