File: pathfinder/pathfinder.kicad_pcb (KiCad board)
At the start: 2 copper layers, 10 parts, among them SW1 SW_Push, SW2 SW_Push, SW3 SW_Push, U1 XIAO-RP2040-DIP

Commit message: Updated
I have done the routing and I am currently working on the 3D stuff
Parts:
- moved SW3 53.5 mm to (79.4, 106.2)
- moved SW1 49.5 mm to (79.4, 67.7)
- moved SW2 49.4 mm to (79.4, 86.9)
- moved R1 6.43 mm to (110.8, 82.7)
- moved R2 5.85 mm to (101.8, 82.8)
- moved R3 5.55 mm to (92.4, 82.8)
- moved U1 4.26 mm to (101.3, 111.8)
- moved D3 3.81 mm to (91.8, 72.5)
- moved D2 3.57 mm to (101.1, 72.2)
- moved D1 3.34 mm to (110.5, 72.3)
Routing:
- net button1: track 0.00 -> 60.1 mm
- net button2: track 0.00 -> 40.5 mm
- net button3: track 0.00 -> 29.6 mm
- net LED1: track 0.00 -> 23.0 mm
- net LED3: track 0.00 -> 15.3 mm
- net LED2: track 0.00 -> 15.0 mm
- net Net-(D2-PadA): track 0.00 -> 10.9 mm
- net Net-(D1-PadA): track 0.00 -> 10.9 mm
- net Net-(D3-PadA): track 0.00 -> 10.6 mm
Other:
- board outline added: 58.2 x 67.3 mm
